File: Lesson 4/EE-Workshop.sch (EAGLE design)
At the start: 1 part

Commit message: Faheema
Parts:
- added C1: (no value), rcl:C-US025-025X050
- added IC1: NE555N, linear:NE555N
- added R1, R3, R9: 1k, rcl:R-US_0207/10
- added R10: 910, rcl:R-US_0207/10
- added R2: 5.2k, rcl:R-US_0207/10
- added R4: 390, rcl:R-US_0207/10
- added R5: 1.5k, rcl:R-US_0207/10
- added R6: 1.3k, rcl:R-US_0207/10
- added R7: 620, rcl:R-US_0207/10
- added R8: 1.1k, rcl:R-US_0207/10
Connections:
- new net 0: BATT.-, C1.2, IC1.GND
- new net N$2: C1.1, IC1.CV
- new net VCC: BATT.+, IC1.R
Other:
- moved on the sheet: BATT
Changed lines of the file:
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@@
 <?xml version="1.0" encoding="utf-8"?>
 <!DOCTYPE eagle SYSTEM "eagle.dtd">
-<eagle version="9.2.2">
+<eagle version="9.4.0">
 <drawing>
 <settings>
@@
 <parts>
 <part name="BATT" library="battery" library_urn="urn:adsk.eagle:library:109" deviceset="AB9V" device="" package3d_urn="urn:adsk.eagle:package:4600/1"/>
+<part name="R2" library="rcl" library_urn="urn:adsk.eagle:library:334" deviceset="R-US_" device="0207/10" package3d_urn="urn:adsk.eagle:package:23491/1" value="5.2k"/>
+<part name="R3" library="rcl" library_urn="urn:adsk.eagle:library:334" deviceset="R-US_" device="0207/10" package3d_urn="urn:adsk.eagle:package:23491/1" value="1k"/>
+<part name="R4" library="rcl" library_urn="urn:adsk.eagle:library:334" deviceset="R-US_" device="0207/10" package3d_urn="urn:adsk.eagle:package:23491/1" value="390"/>
+<part name="IC1" library="linear" library_urn="urn:adsk.eagle:library:262" deviceset="*555" device="N" package3d_urn="urn:adsk.eagle:package:16409/2" technology="NE"/>
+<part name="R5" library="rcl" library_urn="urn:adsk.eagle:library:334" deviceset="R-US_" device="0207/10" package3d_urn="urn:adsk.eagle:package:23491/1" value="1.5k"/>
+<part name="R6" library="rcl" library_urn="urn:adsk.eagle:library:334" deviceset="R-US_" device="0207/10" package3d_urn="urn:adsk.eagle:package:23491/1" value="1.3k"/>
+<part name="R7" library="rcl" library_urn="urn:adsk.eagle:library:334" deviceset="R-US_" device="0207/10" package3d_urn="urn:adsk.eagle:package:23491/1" value="620"/>
+<part name="R8" library="rcl" library_urn="urn:adsk.eagle:library:334" deviceset="R-US_" device="0207/10" package3d_urn="urn:adsk.eagle:package:23491/1" value="1.1k"/>
+<part name="R9" library="rcl" library_urn="urn:adsk.eagle:library:334" deviceset="R-US_" device="0207/10" package3d_urn="urn:adsk.eagle:package:23491/1" value="1k"/>
+<part name="R10" library="rcl" library_urn="urn:adsk.eagle:library:334" deviceset="R-US_" device="0207/10" package3d_urn="urn:adsk.eagle:package:23491/1" value="910"/>
+<part name="R1" library="rcl" library_urn="urn:adsk.eagle:library:334" deviceset="R-US_" device="0207/10" package3d_urn="urn:adsk.eagle:package:23491/1" value="1k"/>
+<part name="X_1" library="ngspice-simulation" library_urn="urn:adsk.eagle:library:527439" deviceset="GND" device=""/>
+<part name="C1" library="rcl" library_urn="urn:adsk.eagle:library:334" deviceset="C-US" device="025-025X050" package3d_urn="urn:adsk.eagle:package:23629/2"/>
+<part name="P+1" library="supply1" library_urn="urn:adsk.eagle:library:371" deviceset="VCC" device=""/>
+<part name="X_2" library="ngspice-simulation" library_urn="urn:adsk.eagle:library:527439" deviceset="GND" device=""/>
+<part name="P+2" library="supply1" library_urn="urn:adsk.eagle:library:371" deviceset="VCC" device=""/>
 </parts>
 <sheets>
@@
 </plain>
 <instances>
-<instance part="BATT" gate="G$1" x="22.86" y="53.34" smashed="yes" rot="R90">
-<attribute name="NAME" x="19.685" y="47.625" size="1.778" layer="95" rot="R90"/>
-<attribute name="VALUE" x="27.94" y="47.625" size="1.778" layer="96" rot="R90"/>
+<instance part="BATT" gate="G$1" x="-91.44" y="38.1" smashed="yes" rot="R90">
+<attribute name="NAME" x="-94.615" y="32.385" size="1.778" layer="95" rot="R90"/>
+<attribute name="VALUE" x="-86.36" y="32.385" size="1.778" layer="96" rot="R90"/>
+</instance>
+<instance part="R2" gate="G$1" x="25.4" y="58.42" smashed="yes">
+<attribute name="NAME" x="21.59" y="59.9186" size="1.778" layer="95"/>
+<attribute name="VALUE" x="21.59" y="55.118" size="1.778" layer="96"/>
+</instance>
+<instance part="R3" gate="G$1" x="17.78" y="66.04" smashed="yes" rot="R270">
+<attribute name="NAME" x="19.2786" y="69.85" size="1.778" layer="95" rot="R270"/>
+<attribute name="VALUE" x="14.478" y="69.85" size="1.778" layer="96" rot="R270"/>
+</instance>
+<instance part="R4" gate="G$1" x="38.1" y="58.42" smashed="yes">
+<attribute name="NAME" x="34.29" y="59.9186" size="1.778" layer="95"/>
+<attribute name="VALUE" x="34.29" y="55.118" size="1.778" layer="96"/>
+</instance>
+<instance part="IC1" gate="A" x="-25.4" y="38.1" smashed="yes">
+<attribute name="NAME" x="-33.02" y="49.022" size="1.778" layer="95"/>
+<attribute name="VALUE" x="-33.02" y="25.273" size="1.778" layer="96"/>
+</instance>
+<instance part="R5" gate="G$1" x="114.3" y="58.42" smashed="yes">
+<attribute name="NAME" x="113.03" y="59.9186" size="1.778" layer="95"/>
+<attribute name="VALUE" x="110.49" y="55.118" size="1.778" layer="96"/>
+</instance>
+<instance part="R6" gate="G$1" x="101.6" y="58.42" smashed="yes">
+<attribute name="NAME" x="97.79" y="59.9186" size="1.778" layer="95"/>
+<attribute name="VALUE" x="97.79" y="55.118" size="1.778" layer="96"/>
+</instance>
+<instance part="R7" gate="G$1" x="88.9" y="58.42" smashed="yes">
+<attribute name="NAME" x="85.09" y="59.9186" size="1.778" layer="95"/>
+<attribute name="VALUE" x="85.09" y="55.118" size="1.778" layer="96"/>
+</instance>
+<instance part="R8" gate="G$1" x="76.2" y="58.42" smashed="yes">
+<attribute name="NAME" x="72.39" y="59.9186" size="1.778" layer="95"/>
+<attribute name="VALUE" x="72.39" y="55.118" size="1.778" layer="96"/>
+</instance>
+<instance part="R9" gate="G$1" x="63.5" y="58.42" smashed="yes">
+<attribute name="NAME" x="59.69" y="59.9186" size="1.778" layer="95"/>
+<attribute name="VALUE" x="59.69" y="55.118" size="1.778" layer="96"/>
+</instance>
+<instance part="R10" gate="G$1" x="50.8" y="58.42" smashed="yes">
+<attribute name="NAME" x="46.99" y="59.9186" size="1.778" layer="95"/>
+<attribute name="VALUE" x="46.99" y="55.118" size="1.778" layer="96"/>
+</instance>
+<instance part="R1" gate="G$1" x="-2.54" y="86.36" smashed="yes">
+<attribute name="NAME" x="-6.35" y="87.8586" size="1.778" layer="95"/>
+<attribute name="VALUE" x="-6.35" y="83.058" size="1.778" layer="96"/>
+</instance>
+<instance part="X_1" gate="G$1" x="-91.44" y="10.16" smashed="yes"/>
+<instance part="C1" gate="G$1" x="-55.88" y="30.48" smashed="yes">
+<attribute name="NAME" x="-54.864" y="31.115" size="1.778" layer="95"/>
+<attribute name="VALUE" x="-54.864" y="26.289" size="1.778" layer="96"/>
+</instance>
+<instance part="P+1" gate="VCC" x="-91.44" y="66.04" smashed="yes">
+<attribute name="VALUE" x="-93.98" y="63.5" size="1.778" layer="96" rot="R90"/>
+</instance>
+<instance part="X_2" gate="G$1" x="-50.8" y="20.32" smashed="yes"/>
+<instance part="P+2" gate="VCC" x="-43.18" y="71.12" smashed="yes">
+<attribute name="VALUE" x="-45.72" y="68.58" size="1.778" layer="96" rot="R90"/>
 </instance>
 </instances>
@@
 </busses>
 <nets>
+<net name="0" class="0">
+<segment>
+<pinref part="BATT" gate="G$1" pin="-"/>
+<wire x1="-91.44" y1="25.4" x2="-91.44" y2="10.16" width="0.1524" layer="91"/>
+<pinref part="X_1" gate="G$1" pin="0"/>
+</segment>
+<segment>
+<pinref part="C1" gate="G$1" pin="2"/>
+<wire x1="-55.88" y1="25.4" x2="-55.88" y2="22.86" width="0.1524" layer="91"/>
+<wire x1="-55.88" y1="22.86" x2="-50.8" y2="22.86" width="0.1524" layer="91"/>
+<pinref part="X_2" gate="G$1" pin="0"/>
+<wire x1="-50.8" y1="22.86" x2="-50.8" y2="20.32" width="0.1524" layer="91"/>
+<wire x1="-50.8" y1="22.86" x2="-45.72" y2="22.86" width="0.1524" layer="91"/>
+<junction x="-50.8" y="22.86"/>
+<wire x1="-45.72" y1="22.86" x2="-45.72" y2="30.48" width="0.1524" layer="91"/>
+<pinref part="IC1" gate="A" pin="GND"/>
+<wire x1="-45.72" y1="30.48" x2="-35.56" y2="30.48" width="0.1524" layer="91"/>
+</segment>
+</net>
+<net name="N$2" class="0">
+<segment>
+<pinref part="IC1" gate="A" pin="CV"/>
+<wire x1="-35.56" y1="35.56" x2="-55.88" y2="35.56" width="0.1524" layer="91"/>
+<pinref part="C1" gate="G$1" pin="1"/>
+<wire x1="-55.88" y1="35.56" x2="-55.88" y2="33.02" width="0.1524" layer="91"/>
+</segment>
+</net>
+<net name="VCC" class="0">
+<segment>
+<pinref part="BATT" gate="G$1" pin="+"/>
+<wire x1="-91.44" y1="50.8" x2="-91.44" y2="63.5" width="0.1524" layer="91"/>
+<pinref part="P+1" gate="VCC" pin="VCC"/>
+</segment>
+<segment>
+<pinref part="IC1" gate="A" pin="R"/>
+<wire x1="-35.56" y1="40.64" x2="-43.18" y2="40.64" width="0.1524" layer="91"/>
+<wire x1="-43.18" y1="40.64" x2="-43.18" y2="68.58" width="0.1524" layer="91"/>
+<pinref part="P+2" gate="VCC" pin="VCC"/>
+</segment>
+</net>
 </nets>
 </sheet>
@@
 packages will not be understood (or retained) with this version.
 </note>
+<note version="8.4" severity="warning">
+Since Version 8.4, EAGLE supports properties for SPICE simulation.
+Probes in schematics and SPICE mapping objects found in parts and library devices
+will not be understood with this version. Update EAGLE to the latest version
+for full support of SPICE simulation.
+</note>
 </compatibility>
